Commit message: update:

File: urdf/camera.urdf.xacro (robot description, xacro)
@@ -4,5 +4,5 @@
 <robot xmlns:xacro="http://www.ros.org/wiki/xacro">
     <xacro:property name="M_PI" value="3.1415926535897931" />
-    <xacro:property name="camera_link" value="0.02" />
+    <xacro:property name="camera_link" value="0.01" />
     <xacro:macro name="camera_model" params="name parent *origin">
       <joint name="${name}_joint" type="fixed">
@@ -45,6 +45,6 @@
             <horizontal_fov>1.256</horizontal_fov>
             <image>
-              <width>640</width>
-              <height>360</height>
+              <width>410</width>
+              <height>308</height>
               <format>R8G8B8</format>
             </image>

File: urdf/turtlebot3_burger.gazebo.xacro (robot description, xacro)
@@ -1,5 +1,5 @@
 <?xml version="1.0"?>
 <robot name="turtlebot3_burger_sim" xmlns:xacro="http://ros.org/wiki/xacro">
-  <xacro:arg name="laser_visual" default="false"/>
+  <xacro:arg name="laser_visual" default="true"/>
   <xacro:arg name="imu_visual"   default="false"/>
   <gazebo reference="base_link">

File: urdf/turtlebot3_burger.urdf.xacro (robot description, xacro)
@@ -141,18 +141,58 @@
   </link>
   <!-- Added by Klaas -->
+  <!-- camera holder -->
+  <joint name="camera_holder_joint" type="fixed">
+    <parent link="base_link"/>
+    <child link="camera_holder"/>
+    <origin xyz="-0.10 0 0.15" rpy="0 0 0"/>
+  </joint>
+  <link name="camera_holder">
+    <visual>
+      <origin xyz="0 0 0.04" rpy="0 0 0"/>
+      <geometry>
+        <box size="0.002 0.01 0.12"/>
+      </geometry>
+    </visual>
+    <collision>
+      <origin xyz="0 0 0.06" rpy="0 0 0"/>
+      <geometry>
+        <box size="0.002 0.01 0.12"/>
+      </geometry>
+    </collision>
+  </link>
+<!--   <joint name="camera_holder_link_joint" type="fixed">
+    <parent link="camera_holder"/>
+    <child link="camera_holder_link"/>
+    <origin xyz="0 0 0.035" rpy="0 0 0"/>
+  </joint> -->
+<!--   <link name="camera_holder_link">
+    <visual>
+      <origin xyz="0.0 0 0" rpy="0 0 0"/>
+      <origin xyz="-0.0615 0 0.24" rpy="0 0 0"/>
+      <geometry>
+        <box size="0.123 0.01 0.002"/>
+      </geometry>
+    </visual>
+ --> <!--     <collision>
+      <origin xyz="0.065 0 0" rpy="0 0 0"/>
+      <geometry>
+        <box size="0.123 0.01 0.002"/>
+      </geometry>
+    </collision> -->
+  <!-- </link> -->
+  <!-- Basic camera -->
+<!--   <xacro:include filename="$(find klaas_robots)/urdf/camera.urdf.xacro" />
+  <xacro:rp_camera name="camera" parent="base_link">
+  <origin xyz="-0.017 0.0 0.24"/>
+  </xacro:rp_camera> -->
   <!-- Kinect -->
-<!--   <xacro:include filename="$(find klaas_robots)/urdf/kinect_camera.urdf.xacro" />
+  <!--   <xacro:include filename="$(find klaas_robots)/urdf/kinect_camera.urdf.xacro" />
   <xacro:kinect_camera name="camera" parent="base_link">
-    <origin xyz="0.15 0.0 0.5" rpy="0 0 0"/>
+    <origin xyz="-0.017 0.0 0.24" rpy="0 0 0"/>
   </xacro:kinect_camera> -->
-  <!-- Basic camera -->
-  <xacro:include filename="$(find klaas_robots)/urdf/camera.urdf.xacro" />
-  <xacro:rp_camera name="camera" parent="base_link">
-  <origin xyz="0.02 0.0 0.11"/>
-  </xacro:rp_camera>
   <!-- Wide angle camera -->
-  <!-- <xacro:include filename="$(find klaas_robots)/urdf/wide_angle_camera.urdf.xacro" />
+  <xacro:include filename="$(find klaas_robots)/urdf/wide_angle_camera.urdf.xacro" />
   <xacro:wide_angle_camera name="camera" parent="base_link">
-  <origin xyz="0.03 0.0 0.11"/>
-  </xacro:wide_angle_camera> -->
+  <origin xyz="-0.017 0.0 0.24"/>
+  </xacro:wide_angle_camera>
 </robot>

File: urdf/wide_angle_camera.urdf.xacro (robot description, xacro)
@@ -42,11 +42,11 @@
         <sensor type="wideanglecamera" name="camera1">
         <!-- <sensor type="camera" name="camera1">-->
-          <update_rate>20.0</update_rate>
+          <update_rate>10.0</update_rate>
           <camera name="head">
-            <!-- 120 degrees horizontal field of view -->
-            <horizontal_fov>2.093</horizontal_fov>
+            <!-- 106 degrees horizontal field of view -->
+            <horizontal_fov>1.849</horizontal_fov>
             <image>
-              <width>640</width>
-              <height>360</height>
+              <width>410</width>
+              <height>308</height>
               <format>R8G8B8</format>
             </image>
